File: PCBs/Chocolate.kicad_pcb (KiCad board)
At the start: 2 copper layers, 100 x 100 mm, 86 parts, among them J1 163-179PH-EX, J10 Conn_01x01_Male, J11 Conn_01x01_Male, J12 Conn_01x01_Male, J13 Conn_01x01_Male, J14 Conn_01x01_Male, J15 Conn_01x01_Male, J16 Screw_Terminal_01x04, J17 Screw_Terminal_01x04, J18 09185166324, J19 Conn_01x01_Male, J2 Conn_01x01_Male, J20 Conn_01x01_Male, J21 Conn_01x01_Male, J22 Conn_01x01_Male, J23 Conn_01x01_Male, J24 Conn_01x01_Male, J25 Conn_01x01_Male, J26 Conn_01x01_Male, J27 Screw_Terminal_01x04, J28 Screw_Terminal_01x04, J29 09185166324, J3 Conn_01x01_Male, J30 09185166324, J31 09185166324, J32 09185166324, J33 09185166324, J4 Conn_01x01_Male, J5 Conn_01x01_Male, J6 Conn_01x01_Male, J7 Conn_01x01_Male, J8 Conn_01x01_Male, J9 Conn_01x01_Male, U1 L7805

Commit message: Regulator goes to sleep
Use a different footprint for the L7805
Parts:
- U1: footprint Package_TO_SOT_THT:TO-220-3_Vertical -> Package_TO_SOT_THT:TO-220-3_Horizontal_TabDown
- moved C1 20.6 mm to (36.5, -48.4), turned to 0 degrees
- moved C2 16.2 mm to (51.0, -48.4), turned to 0 degrees
- moved C4 10.3 mm to (29.2, -48.4)
- moved C3 6.00 mm to (43.8, -48.4)
- moved U1 2.03 mm to (36.6, -34.0)
- moved REF** 1.50 mm to (3.30, -31.5)
- moved REF** 1.50 mm to (3.30, 28.5)
- moved REF** 1.50 mm to (53.3, -31.5)
- moved REF** 1.50 mm to (53.3, 28.5)
Routing:
- net +5V: track 304.2 -> 293.2 mm
- net -12V: track 275.4 -> 280.5 mm
- net +12V: track 387.7 -> 383.1 mm

Commit message: Mostly cosmetics
Parts:
- renumbered C4 to C1, C1 to C2, C2 to C4, D3 to D2, D2 to D3
Routing:
- net +12V: track 383.1 -> 388.9 mm
- net +5V: track 293.2 -> 294.4 mm
- net -12V: track 280.5 -> 281.1 mm
