File: PCBs/Chocolate.kicad_sch (KiCad schematic)
At the start: 48 parts, among them J1 163-179PH-EX, J10 Conn_01x01_Male, J11 Conn_01x01_Male, J12 Conn_01x01_Male, J13 Conn_01x01_Male, J14 Conn_01x01_Male, J15 Conn_01x01_Male, J16 Screw_Terminal_01x04, J17 Screw_Terminal_01x04, J18 09185166324, J19 Conn_01x01_Male, J2 Conn_01x01_Male, J20 Conn_01x01_Male, J21 Conn_01x01_Male, J22 Conn_01x01_Male, J23 Conn_01x01_Male, J24 Conn_01x01_Male, J25 Conn_01x01_Male, J26 Conn_01x01_Male, J27 Screw_Terminal_01x04, J28 Screw_Terminal_01x04, J29 09185166324, J3 Conn_01x01_Male, J30 09185166324, J31 09185166324, J32 09185166324, J33 09185166324, J4 Conn_01x01_Male, J5 Conn_01x01_Male, J6 Conn_01x01_Male, J7 Conn_01x01_Male, J8 Conn_01x01_Male, J9 Conn_01x01_Male, U1 L7805

Commit message: Regulator goes to sleep
Use a different footprint for the L7805
Parts:
- U1: footprint Package_TO_SOT_THT:TO-220-3_Vertical -> Package_TO_SOT_THT:TO-220-3_Horizontal_TabDown
Changed lines of the file:
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@@
     (property "Reference" "U1" (id 0) (at 229.235 20.1635 0))
     (property "Value" "L7805" (id 1) (at 229.235 22.9386 0))
-    (property "Footprint" "Package_TO_SOT_THT:TO-220-3_Vertical" (id 2) (at 229.87 29.845 0)
+    (property "Footprint" "Package_TO_SOT_THT:TO-220-3_Horizontal_TabDown" (id 2) (at 229.87 29.845 0)
       (effects (font (size 1.27 1.27) italic) (justify left) hide)
     )
@@
     )
     (path "/fbc71af7-de54-4238-9761-e2dd07bc84ed"
-      (reference "U1") (unit 1) (value "L7805") (footprint "Package_TO_SOT_THT:TO-220-3_Vertical")
+      (reference "U1") (unit 1) (value "L7805") (footprint "Package_TO_SOT_THT:TO-220-3_Horizontal_TabDown")
     )
   )

Commit message: Mostly cosmetics
Parts:
- renumbered C4 to C1, C1 to C2, C2 to C4, D3 to D2, D2 to D3
Changed lines of the file:
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@@
   (symbol (lib_id "Device:C") (at 217.805 29.845 0) (unit 1)
     (in_bom yes) (on_board yes)
-    (property "Reference" "C1" (id 0) (at 208.915 29.845 0)
+    (property "Reference" "C2" (id 0) (at 208.915 29.845 0)
       (effects (font (size 1.27 1.27)) (justify left))
     )
@@
   (symbol (lib_id "Device:C") (at 240.665 29.845 0) (unit 1)
     (in_bom yes) (on_board yes) (fields_autoplaced)
-    (property "Reference" "C2" (id 0) (at 243.586 28.9365 0)
+    (property "Reference" "C4" (id 0) (at 243.586 28.9365 0)
       (effects (font (size 1.27 1.27)) (justify left))
     )
@@
   (symbol (lib_id "Device:LED") (at 139.065 92.71 0) (unit 1)
     (in_bom yes) (on_board yes) (fields_autoplaced)
-    (property "Reference" "D2" (id 0) (at 137.4775 87.4735 0))
+    (property "Reference" "D3" (id 0) (at 137.4775 87.4735 0))
     (property "Value" "LED" (id 1) (at 137.4775 90.2486 0))
     (property "Footprint" "LED_THT:LED_D5.0mm" (id 2) (at 139.065 92.71 0)
@@
   (symbol (lib_id "Device:C") (at 269.24 31.75 0) (unit 1)
     (in_bom yes) (on_board yes)
-    (property "Reference" "C4" (id 0) (at 271.78 31.75 0)
+    (property "Reference" "C1" (id 0) (at 271.78 31.75 0)
       (effects (font (size 1.27 1.27)) (justify left))
     )
@@
   (symbol (lib_id "Device:LED") (at 147.955 102.87 180) (unit 1)
     (in_bom yes) (on_board yes) (fields_autoplaced)
-    (property "Reference" "D3" (id 0) (at 149.5425 96.7445 0))
+    (property "Reference" "D2" (id 0) (at 149.5425 96.7445 0))
     (property "Value" "LED" (id 1) (at 149.5425 99.5196 0))
     (property "Footprint" "LED_THT:LED_D5.0mm" (id 2) (at 147.955 102.87 0)
@@
       (reference "#PWR05") (unit 1) (value "GND") (footprint "")
     )
+    (path "/941cdffe-2cb5-499b-8328-8baccc4eb37f"
+      (reference "C1") (unit 1) (value "330n") (footprint "Capacitor_THT:C_Disc_D5.0mm_W2.5mm_P5.00mm")
+    )
     (path "/1640c815-f26e-47fb-afd0-e5fad0a2ba7c"
-      (reference "C1") (unit 1) (value "330n") (footprint "Capacitor_THT:C_Disc_D5.0mm_W2.5mm_P5.00mm")
-    )
-    (path "/3fb484cb-cd4c-4513-8341-534ee5f71206"
-      (reference "C2") (unit 1) (value "100n") (footprint "Capacitor_THT:C_Disc_D5.0mm_W2.5mm_P5.00mm")
+      (reference "C2") (unit 1) (value "330n") (footprint "Capacitor_THT:C_Disc_D5.0mm_W2.5mm_P5.00mm")
     )
     (path "/74315917-dce5-4769-a3b7-a2d2033698d9"
       (reference "C3") (unit 1) (value "330n") (footprint "Capacitor_THT:C_Disc_D5.0mm_W2.5mm_P5.00mm")
     )
-    (path "/941cdffe-2cb5-499b-8328-8baccc4eb37f"
-      (reference "C4") (unit 1) (value "330n") (footprint "Capacitor_THT:C_Disc_D5.0mm_W2.5mm_P5.00mm")
+    (path "/3fb484cb-cd4c-4513-8341-534ee5f71206"
+      (reference "C4") (unit 1) (value "100n") (footprint "Capacitor_THT:C_Disc_D5.0mm_W2.5mm_P5.00mm")
     )
     (path "/b3a8f536-9ead-4b4b-ac82-179916ddcc67"
       (reference "D1") (unit 1) (value "LED") (footprint "LED_THT:LED_D5.0mm")
     )
+    (path "/bda5bd79-46d0-470f-978e-3a8f830bb866"
+      (reference "D2") (unit 1) (value "LED") (footprint "LED_THT:LED_D5.0mm")
+    )
     (path "/720c1001-1a44-4a0c-8694-00b65e09e7d8"
-      (reference "D2") (unit 1) (value "LED") (footprint "LED_THT:LED_D5.0mm")
-    )
-    (path "/bda5bd79-46d0-470f-978e-3a8f830bb866"
       (reference "D3") (unit 1) (value "LED") (footprint "LED_THT:LED_D5.0mm")
     )
